Commit message: adding location offset to urdfs

File: interbotix_arm_robot_server/urdf/px100.urdf.xacro (robot description, xacro)
@@ -9,4 +9,18 @@
   <xacro:arg name="external_urdf_loc" default=""/>
   <xacro:arg name="load_gazebo_configs" default="false"/>
+  <xacro:arg name="x" default="0.0"/>
+  <xacro:arg name="y" default="0.0"/>
+  <xacro:arg name="z" default="0.0"/>
+  <xacro:arg name="roll" default="0.0"/>
+  <xacro:arg name="pitch" default="0.0"/>
+  <xacro:arg name="yaw" default="0.0"/>
+  <!-- rgbd camera arguments -->
+  <xacro:arg name="camera1_gazebo" default="False"/>
+  <xacro:arg name="camera1_link_x" default="0.0"/>
+  <xacro:arg name="camera1_link_y" default="0.0"/>
+  <xacro:arg name="camera1_link_z" default="0.0"/>
+  <xacro:arg name="camera1_link_roll" default="0.0"/>
+  <xacro:arg name="camera1_link_pitch" default="0.0"/>
+  <xacro:arg name="camera1_link_yaw" default="0.0"/>
   <xacro:property name="urdf_loc" value="$(arg external_urdf_loc)"/>
   <xacro:property name="pi_offset" value="0.00001"/>
@@ -88,4 +102,5 @@
       <parent link="world"/>
       <child link="$(arg robot_name)/$(arg base_link_frame)"/>
+      <origin xyz="$(arg x) $(arg y) $(arg z)" rpy="$(arg roll) $(arg pitch) $(arg yaw)" />
     </joint>
   </xacro:if>
@@ -472,3 +487,14 @@
     <xacro:include filename="${urdf_loc}"/>
   </xacro:if>
+  <!-- simulated rgbd camera include -->
+  <xacro:if value="$(arg camera1_gazebo)">
+    <xacro:include filename="$(find scene_perception)/urdf/rgbd_camera_macro.xacro"/>
+    <xacro:rgbd_camera_gazebo camera_name="camera1"/>
+    <joint name="camera1_joint" type="fixed">
+      <parent link="world"/>
+      <child link="camera1_link"/>
+      <origin xyz="$(arg camera1_link_x) $(arg camera1_link_y) $(arg camera1_link_z)"
+        rpy="$(arg camera1_link_roll) $(arg camera1_link_pitch) $(arg camera1_link_yaw)" />
+    </joint>
+  </xacro:if>
 </robot>

File: interbotix_arm_robot_server/urdf/px150.urdf.xacro (robot description, xacro)
@@ -9,4 +9,18 @@
   <xacro:arg name="external_urdf_loc" default=""/>
   <xacro:arg name="load_gazebo_configs" default="false"/>
+  <xacro:arg name="x" default="0.0"/>
+  <xacro:arg name="y" default="0.0"/>
+  <xacro:arg name="z" default="0.0"/>
+  <xacro:arg name="roll" default="0.0"/>
+  <xacro:arg name="pitch" default="0.0"/>
+  <xacro:arg name="yaw" default="0.0"/>
+  <!-- rgbd camera arguments -->
+  <xacro:arg name="camera1_gazebo" default="False"/>
+  <xacro:arg name="camera1_link_x" default="0.0"/>
+  <xacro:arg name="camera1_link_y" default="0.0"/>
+  <xacro:arg name="camera1_link_z" default="0.0"/>
+  <xacro:arg name="camera1_link_roll" default="0.0"/>
+  <xacro:arg name="camera1_link_pitch" default="0.0"/>
+  <xacro:arg name="camera1_link_yaw" default="0.0"/>
   <xacro:property name="urdf_loc" value="$(arg external_urdf_loc)"/>
   <xacro:property name="pi_offset" value="0.00001"/>
@@ -104,4 +118,5 @@
       <parent link="world"/>
       <child link="$(arg robot_name)/$(arg base_link_frame)"/>
+      <origin xyz="$(arg x) $(arg y) $(arg z)" rpy="$(arg roll) $(arg pitch) $(arg yaw)" />
     </joint>
   </xacro:if>
@@ -525,3 +540,14 @@
     <xacro:include filename="${urdf_loc}"/>
   </xacro:if>
+  <!-- simulated rgbd camera include -->
+  <xacro:if value="$(arg camera1_gazebo)">
+    <xacro:include filename="$(find scene_perception)/urdf/rgbd_camera_macro.xacro"/>
+    <xacro:rgbd_camera_gazebo camera_name="camera1"/>
+    <joint name="camera1_joint" type="fixed">
+      <parent link="world"/>
+      <child link="camera1_link"/>
+      <origin xyz="$(arg camera1_link_x) $(arg camera1_link_y) $(arg camera1_link_z)"
+        rpy="$(arg camera1_link_roll) $(arg camera1_link_pitch) $(arg camera1_link_yaw)" />
+    </joint>
+  </xacro:if>
 </robot>

File: interbotix_arm_robot_server/urdf/rx200.urdf.xacro (robot description, xacro)
@@ -9,4 +9,18 @@
   <xacro:arg name="external_urdf_loc" default=""/>
   <xacro:arg name="load_gazebo_configs" default="false"/>
+  <xacro:arg name="x" default="0.0"/>
+  <xacro:arg name="y" default="0.0"/>
+  <xacro:arg name="z" default="0.0"/>
+  <xacro:arg name="roll" default="0.0"/>
+  <xacro:arg name="pitch" default="0.0"/>
+  <xacro:arg name="yaw" default="0.0"/>
+  <!-- rgbd camera arguments -->
+  <xacro:arg name="camera1_gazebo" default="False"/>
+  <xacro:arg name="camera1_link_x" default="0.0"/>
+  <xacro:arg name="camera1_link_y" default="0.0"/>
+  <xacro:arg name="camera1_link_z" default="0.0"/>
+  <xacro:arg name="camera1_link_roll" default="0.0"/>
+  <xacro:arg name="camera1_link_pitch" default="0.0"/>
+  <xacro:arg name="camera1_link_yaw" default="0.0"/>
   <xacro:property name="urdf_loc" value="$(arg external_urdf_loc)"/>
   <xacro:property name="pi_offset" value="0.00001"/>
@@ -104,4 +118,5 @@
       <parent link="world"/>
       <child link="$(arg robot_name)/$(arg base_link_frame)"/>
+      <origin xyz="$(arg x) $(arg y) $(arg z)" rpy="$(arg roll) $(arg pitch) $(arg yaw)" />
     </joint>
   </xacro:if>
@@ -525,3 +540,14 @@
     <xacro:include filename="${urdf_loc}"/>
   </xacro:if>
+  <!-- simulated rgbd camera include -->
+  <xacro:if value="$(arg camera1_gazebo)">
+    <xacro:include filename="$(find scene_perception)/urdf/rgbd_camera_macro.xacro"/>
+    <xacro:rgbd_camera_gazebo camera_name="camera1"/>
+    <joint name="camera1_joint" type="fixed">
+      <parent link="world"/>
+      <child link="camera1_link"/>
+      <origin xyz="$(arg camera1_link_x) $(arg camera1_link_y) $(arg camera1_link_z)"
+        rpy="$(arg camera1_link_roll) $(arg camera1_link_pitch) $(arg camera1_link_yaw)" />
+    </joint>
+  </xacro:if>
 </robot>

File: interbotix_arm_robot_server/urdf/vx250.urdf.xacro (robot description, xacro)
@@ -9,4 +9,18 @@
   <xacro:arg name="external_urdf_loc" default=""/>
   <xacro:arg name="load_gazebo_configs" default="false"/>
+  <xacro:arg name="x" default="0.0"/>
+  <xacro:arg name="y" default="0.0"/>
+  <xacro:arg name="z" default="0.0"/>
+  <xacro:arg name="roll" default="0.0"/>
+  <xacro:arg name="pitch" default="0.0"/>
+  <xacro:arg name="yaw" default="0.0"/>
+  <!-- rgbd camera arguments -->
+  <xacro:arg name="camera1_gazebo" default="False"/>
+  <xacro:arg name="camera1_link_x" default="0.0"/>
+  <xacro:arg name="camera1_link_y" default="0.0"/>
+  <xacro:arg name="camera1_link_z" default="0.0"/>
+  <xacro:arg name="camera1_link_roll" default="0.0"/>
+  <xacro:arg name="camera1_link_pitch" default="0.0"/>
+  <xacro:arg name="camera1_link_yaw" default="0.0"/>
   <xacro:property name="urdf_loc" value="$(arg external_urdf_loc)"/>
   <xacro:property name="pi_offset" value="0.00001"/>
@@ -104,4 +118,5 @@
       <parent link="world"/>
       <child link="$(arg robot_name)/$(arg base_link_frame)"/>
+      <origin xyz="$(arg x) $(arg y) $(arg z)" rpy="$(arg roll) $(arg pitch) $(arg yaw)" />
     </joint>
   </xacro:if>
@@ -525,3 +540,14 @@
     <xacro:include filename="${urdf_loc}"/>
   </xacro:if>
+  <!-- simulated rgbd camera include -->
+  <xacro:if value="$(arg camera1_gazebo)">
+    <xacro:include filename="$(find scene_perception)/urdf/rgbd_camera_macro.xacro"/>
+    <xacro:rgbd_camera_gazebo camera_name="camera1"/>
+    <joint name="camera1_joint" type="fixed">
+      <parent link="world"/>
+      <child link="camera1_link"/>
+      <origin xyz="$(arg camera1_link_x) $(arg camera1_link_y) $(arg camera1_link_z)"
+        rpy="$(arg camera1_link_roll) $(arg camera1_link_pitch) $(arg camera1_link_yaw)" />
+    </joint>
+  </xacro:if>
 </robot>

File: interbotix_arm_robot_server/urdf/vx300.urdf.xacro (robot description, xacro)
@@ -9,4 +9,18 @@
   <xacro:arg name="external_urdf_loc" default=""/>
   <xacro:arg name="load_gazebo_configs" default="false"/>
+  <xacro:arg name="x" default="0.0"/>
+  <xacro:arg name="y" default="0.0"/>
+  <xacro:arg name="z" default="0.0"/>
+  <xacro:arg name="roll" default="0.0"/>
+  <xacro:arg name="pitch" default="0.0"/>
+  <xacro:arg name="yaw" default="0.0"/>
+  <!-- rgbd camera arguments -->
+  <xacro:arg name="camera1_gazebo" default="False"/>
+  <xacro:arg name="camera1_link_x" default="0.0"/>
+  <xacro:arg name="camera1_link_y" default="0.0"/>
+  <xacro:arg name="camera1_link_z" default="0.0"/>
+  <xacro:arg name="camera1_link_roll" default="0.0"/>
+  <xacro:arg name="camera1_link_pitch" default="0.0"/>
+  <xacro:arg name="camera1_link_yaw" default="0.0"/>
   <xacro:property name="urdf_loc" value="$(arg external_urdf_loc)"/>
   <xacro:property name="pi_offset" value="0.00001"/>
@@ -104,4 +118,5 @@
       <parent link="world"/>
       <child link="$(arg robot_name)/$(arg base_link_frame)"/>
+      <origin xyz="$(arg x) $(arg y) $(arg z)" rpy="$(arg roll) $(arg pitch) $(arg yaw)" />
     </joint>
   </xacro:if>
@@ -525,3 +540,14 @@
     <xacro:include filename="${urdf_loc}"/>
   </xacro:if>
+  <!-- simulated rgbd camera include -->
+  <xacro:if value="$(arg camera1_gazebo)">
+    <xacro:include filename="$(find scene_perception)/urdf/rgbd_camera_macro.xacro"/>
+    <xacro:rgbd_camera_gazebo camera_name="camera1"/>
+    <joint name="camera1_joint" type="fixed">
+      <parent link="world"/>
+      <child link="camera1_link"/>
+      <origin xyz="$(arg camera1_link_x) $(arg camera1_link_y) $(arg camera1_link_z)"
+        rpy="$(arg camera1_link_roll) $(arg camera1_link_pitch) $(arg camera1_link_yaw)" />
+    </joint>
+  </xacro:if>
 </robot>

File: interbotix_arm_robot_server/urdf/vx300s.urdf.xacro (robot description, xacro)
@@ -9,4 +9,18 @@
   <xacro:arg name="external_urdf_loc" default=""/>
   <xacro:arg name="load_gazebo_configs" default="false"/>
+  <xacro:arg name="x" default="0.0"/>
+  <xacro:arg name="y" default="0.0"/>
+  <xacro:arg name="z" default="0.0"/>
+  <xacro:arg name="roll" default="0.0"/>
+  <xacro:arg name="pitch" default="0.0"/>
+  <xacro:arg name="yaw" default="0.0"/>
+  <!-- rgbd camera arguments -->
+  <xacro:arg name="camera1_gazebo" default="False"/>
+  <xacro:arg name="camera1_link_x" default="0.0"/>
+  <xacro:arg name="camera1_link_y" default="0.0"/>
+  <xacro:arg name="camera1_link_z" default="0.0"/>
+  <xacro:arg name="camera1_link_roll" default="0.0"/>
+  <xacro:arg name="camera1_link_pitch" default="0.0"/>
+  <xacro:arg name="camera1_link_yaw" default="0.0"/>
   <xacro:property name="urdf_loc" value="$(arg external_urdf_loc)"/>
   <xacro:property name="pi_offset" value="0.00001"/>
@@ -120,4 +134,5 @@
       <parent link="world"/>
       <child link="$(arg robot_name)/$(arg base_link_frame)"/>
+      <origin xyz="$(arg x) $(arg y) $(arg z)" rpy="$(arg roll) $(arg pitch) $(arg yaw)" />
     </joint>
   </xacro:if>
@@ -578,3 +593,14 @@
     <xacro:include filename="${urdf_loc}"/>
   </xacro:if>
+  <!-- simulated rgbd camera include -->
+  <xacro:if value="$(arg camera1_gazebo)">
+    <xacro:include filename="$(find scene_perception)/urdf/rgbd_camera_macro.xacro"/>
+    <xacro:rgbd_camera_gazebo camera_name="camera1"/>
+    <joint name="camera1_joint" type="fixed">
+      <parent link="world"/>
+      <child link="camera1_link"/>
+      <origin xyz="$(arg camera1_link_x) $(arg camera1_link_y) $(arg camera1_link_z)"
+        rpy="$(arg camera1_link_roll) $(arg camera1_link_pitch) $(arg camera1_link_yaw)" />
+    </joint>
+  </xacro:if>
 </robot>

File: interbotix_arm_robot_server/urdf/wx200.urdf.xacro (robot description, xacro)
@@ -9,4 +9,18 @@
   <xacro:arg name="external_urdf_loc" default=""/>
   <xacro:arg name="load_gazebo_configs" default="false"/>
+  <xacro:arg name="x" default="0.0"/>
+  <xacro:arg name="y" default="0.0"/>
+  <xacro:arg name="z" default="0.0"/>
+  <xacro:arg name="roll" default="0.0"/>
+  <xacro:arg name="pitch" default="0.0"/>
+  <xacro:arg name="yaw" default="0.0"/>
+  <!-- rgbd camera arguments -->
+  <xacro:arg name="camera1_gazebo" default="False"/>
+  <xacro:arg name="camera1_link_x" default="0.0"/>
+  <xacro:arg name="camera1_link_y" default="0.0"/>
+  <xacro:arg name="camera1_link_z" default="0.0"/>
+  <xacro:arg name="camera1_link_roll" default="0.0"/>
+  <xacro:arg name="camera1_link_pitch" default="0.0"/>
+  <xacro:arg name="camera1_link_yaw" default="0.0"/>
   <xacro:property name="urdf_loc" value="$(arg external_urdf_loc)"/>
   <xacro:property name="pi_offset" value="0.00001"/>
@@ -104,4 +118,5 @@
       <parent link="world"/>
       <child link="$(arg robot_name)/$(arg base_link_frame)"/>
+      <origin xyz="$(arg x) $(arg y) $(arg z)" rpy="$(arg roll) $(arg pitch) $(arg yaw)" />
     </joint>
   </xacro:if>
@@ -525,3 +540,14 @@
     <xacro:include filename="${urdf_loc}"/>
   </xacro:if>
+  <!-- simulated rgbd camera include -->
+  <xacro:if value="$(arg camera1_gazebo)">
+    <xacro:include filename="$(find scene_perception)/urdf/rgbd_camera_macro.xacro"/>
+    <xacro:rgbd_camera_gazebo camera_name="camera1"/>
+    <joint name="camera1_joint" type="fixed">
+      <parent link="world"/>
+      <child link="camera1_link"/>
+      <origin xyz="$(arg camera1_link_x) $(arg camera1_link_y) $(arg camera1_link_z)"
+        rpy="$(arg camera1_link_roll) $(arg camera1_link_pitch) $(arg camera1_link_yaw)" />
+    </joint>
+  </xacro:if>
 </robot>

File: interbotix_arm_robot_server/urdf/wx250.urdf.xacro (robot description, xacro)
@@ -9,4 +9,18 @@
   <xacro:arg name="external_urdf_loc" default=""/>
   <xacro:arg name="load_gazebo_configs" default="false"/>
+  <xacro:arg name="x" default="0.0"/>
+  <xacro:arg name="y" default="0.0"/>
+  <xacro:arg name="z" default="0.0"/>
+  <xacro:arg name="roll" default="0.0"/>
+  <xacro:arg name="pitch" default="0.0"/>
+  <xacro:arg name="yaw" default="0.0"/>
+  <!-- rgbd camera arguments -->
+  <xacro:arg name="camera1_gazebo" default="False"/>
+  <xacro:arg name="camera1_link_x" default="0.0"/>
+  <xacro:arg name="camera1_link_y" default="0.0"/>
+  <xacro:arg name="camera1_link_z" default="0.0"/>
+  <xacro:arg name="camera1_link_roll" default="0.0"/>
+  <xacro:arg name="camera1_link_pitch" default="0.0"/>
+  <xacro:arg name="camera1_link_yaw" default="0.0"/>
   <xacro:property name="urdf_loc" value="$(arg external_urdf_loc)"/>
   <xacro:property name="pi_offset" value="0.00001"/>
@@ -104,4 +118,5 @@
       <parent link="world"/>
       <child link="$(arg robot_name)/$(arg base_link_frame)"/>
+      <origin xyz="$(arg x) $(arg y) $(arg z)" rpy="$(arg roll) $(arg pitch) $(arg yaw)" />
     </joint>
   </xacro:if>
@@ -525,3 +540,14 @@
     <xacro:include filename="${urdf_loc}"/>
   </xacro:if>
+  <!-- simulated rgbd camera include -->
+  <xacro:if value="$(arg camera1_gazebo)">
+    <xacro:include filename="$(find scene_perception)/urdf/rgbd_camera_macro.xacro"/>
+    <xacro:rgbd_camera_gazebo camera_name="camera1"/>
+    <joint name="camera1_joint" type="fixed">
+      <parent link="world"/>
+      <child link="camera1_link"/>
+      <origin xyz="$(arg camera1_link_x) $(arg camera1_link_y) $(arg camera1_link_z)"
+        rpy="$(arg camera1_link_roll) $(arg camera1_link_pitch) $(arg camera1_link_yaw)" />
+    </joint>
+  </xacro:if>
 </robot>

File: interbotix_arm_robot_server/urdf/wx250s.urdf.xacro (robot description, xacro)
@@ -9,4 +9,18 @@
   <xacro:arg name="external_urdf_loc" default=""/>
   <xacro:arg name="load_gazebo_configs" default="false"/>
+  <xacro:arg name="x" default="0.0"/>
+  <xacro:arg name="y" default="0.0"/>
+  <xacro:arg name="z" default="0.0"/>
+  <xacro:arg name="roll" default="0.0"/>
+  <xacro:arg name="pitch" default="0.0"/>
+  <xacro:arg name="yaw" default="0.0"/>
+  <!-- rgbd camera arguments -->
+  <xacro:arg name="camera1_gazebo" default="False"/>
+  <xacro:arg name="camera1_link_x" default="0.0"/>
+  <xacro:arg name="camera1_link_y" default="0.0"/>
+  <xacro:arg name="camera1_link_z" default="0.0"/>
+  <xacro:arg name="camera1_link_roll" default="0.0"/>
+  <xacro:arg name="camera1_link_pitch" default="0.0"/>
+  <xacro:arg name="camera1_link_yaw" default="0.0"/>
   <xacro:property name="urdf_loc" value="$(arg external_urdf_loc)"/>
   <xacro:property name="pi_offset" value="0.00001"/>
@@ -107,4 +121,5 @@
       <parent link="world"/>
       <child link="$(arg robot_name)/$(arg base_link_frame)"/>
+      <origin xyz="$(arg x) $(arg y) $(arg z)" rpy="$(arg roll) $(arg pitch) $(arg yaw)" />
     </joint>
   </xacro:if>
@@ -565,3 +580,14 @@
     <xacro:include filename="${urdf_loc}"/>
   </xacro:if>
+  <!-- simulated rgbd camera include -->
+  <xacro:if value="$(arg camera1_gazebo)">
+    <xacro:include filename="$(find scene_perception)/urdf/rgbd_camera_macro.xacro"/>
+    <xacro:rgbd_camera_gazebo camera_name="camera1"/>
+    <joint name="camera1_joint" type="fixed">
+      <parent link="world"/>
+      <child link="camera1_link"/>
+      <origin xyz="$(arg camera1_link_x) $(arg camera1_link_y) $(arg camera1_link_z)"
+        rpy="$(arg camera1_link_roll) $(arg camera1_link_pitch) $(arg camera1_link_yaw)" />
+    </joint>
+  </xacro:if>
 </robot>
