Commit message: interbotix arm done

File: interbotix_arm_robot_server/urdf/control.urdf.xacro (robot description, xacro)
@@ -19,4 +19,7 @@
         <plugin>gazebo_ros2_control/GazeboSystem</plugin>
       </xacro:if>
+      <xacro:if value="${hardware_type == 'gz_ign'}">
+        <plugin>ign_ros2_control/IgnitionSystem</plugin>
+      </xacro:if>
     </hardware>
     <joint name="waist">
@@ -25,5 +28,7 @@
         <param name="max">"${waist_limit_upper}"</param>
       </command_interface>
+      <command_interface name="velocity"/>
       <state_interface name="position"/>
+      <state_interface name="velocity"/>
     </joint>
     <joint name="shoulder">
@@ -32,5 +37,7 @@
         <param name="max">"${shoulder_limit_upper}"</param>
       </command_interface>
+      <command_interface name="velocity"/>
       <state_interface name="position"/>
+      <state_interface name="velocity"/>
     </joint>
     <joint name="elbow">
@@ -39,5 +46,7 @@
         <param name="max">"${elbow_limit_upper}"</param>
       </command_interface>
+      <command_interface name="velocity"/>
       <state_interface name="position"/>
+      <state_interface name="velocity"/>
     </joint>
     <xacro:if value="${dof >= 6}">
@@ -47,5 +56,7 @@
           <param name="max">"${forearm_roll_limit_upper}"</param>
         </command_interface>
+        <command_interface name="velocity"/>
         <state_interface name="position"/>
+        <state_interface name="velocity"/>
       </joint>
     </xacro:if>
@@ -55,5 +66,7 @@
         <param name="max">"${wrist_angle_limit_upper}"</param>
       </command_interface>
+      <command_interface name="velocity"/>
       <state_interface name="position"/>
+      <state_interface name="velocity"/>
     </joint>
     <xacro:if value="${dof >= 5}">
@@ -63,9 +76,11 @@
           <param name="max">"${wrist_rotate_limit_upper}"</param>
         </command_interface>
+        <command_interface name="velocity"/>
         <state_interface name="position"/>
+        <state_interface name="velocity"/>
       </joint>
     </xacro:if>
     <xacro:if value="$(arg use_gripper)">
-      <xacro:if value="${hardware_type in ('fake', 'gz_classic')}">
+      <xacro:if value="${hardware_type in ('fake', 'gz_classic', 'gz_ign')}">
         <joint name="gripper">
           <command_interface name="position"/>
@@ -81,5 +96,5 @@
           <state_interface name="position"/>
         </joint>
-        <xacro:if value="${hardware_type == 'gz_classic'}">
+        <xacro:if value="${hardware_type in ('gz_classic', 'gz_ign')}">
           <joint name="right_finger">
             <!-- <param name="mimic">left_finger</param>

File: interbotix_arm_robot_server/urdf/mobile_px100.urdf.xacro (robot description, xacro)
@@ -16,7 +16,10 @@
   <xacro:arg name="external_urdf_loc"               default=""/>
   <xacro:arg name="hardware_type"                   default="actual"/>
+  <xacro:arg name="sim_ignition"                    default="true"/>
+  <xacro:arg name="simulation_controllers"          default="" />
   <xacro:property name="mesh_directory"             value="package://interbotix_xsarm_descriptions/meshes/${robot_model}_meshes"/>
   <xacro:property name="urdf_loc"                   value="$(arg external_urdf_loc)"/>
   <xacro:property name="hardware_type"              value="$(arg hardware_type)"/>
+  <xacro:property name="sim_ignition"               value="$(arg sim_ignition)"/>
   <xacro:property name="pi_offset"                  value="0.00001"/>
   <xacro:property name="waist_limit_effort"         value="1"/>
@@ -596,8 +599,19 @@
     </xacro:if> <!-- show_gripper_bar -->
   </xacro:if> <!-- use_gripper -->
-  <xacro:include filename="$(find interbotix_xsarm_descriptions)/urdf/control.urdf.xacro"/>
+  <xacro:include filename="$(find interbotix_arm_robot_server)/urdf/control.urdf.xacro"/>
   <xacro:include filename="$(find interbotix_xsarm_descriptions)/urdf/gazebo_configs.urdf.xacro"/>
   <xacro:if value="${hardware_type == 'gz_classic'}">
     <xacro:gazebo_configs/>
+  </xacro:if>
+  <xacro:if value="$(arg sim_ignition)">
+    <!-- Gazebo plugins -->
+    <gazebo reference="world">
+    </gazebo>
+    <gazebo>
+      <plugin filename="libign_ros2_control-system.so" name="ign_ros2_control::IgnitionROS2ControlPlugin">
+        <parameters>$(arg simulation_controllers)</parameters>
+        <controller_manager_node_name>$(arg tf_prefix)controller_manager</controller_manager_node_name>
+      </plugin>
+    </gazebo>
   </xacro:if>
   <xacro:if value="${urdf_loc != ''}">

File: interbotix_arm_robot_server/urdf/mobile_wx200.urdf.xacro (robot description, xacro)
@@ -16,7 +16,10 @@
   <xacro:arg name="external_urdf_loc"               default=""/>
   <xacro:arg name="hardware_type"                   default="actual"/>
+  <xacro:arg name="sim_ignition"                    default="true"/>
+  <xacro:arg name="simulation_controllers"          default="" />
   <xacro:property name="mesh_directory"             value="package://interbotix_xsarm_descriptions/meshes/${robot_model}_meshes"/>
   <xacro:property name="urdf_loc"                   value="$(arg external_urdf_loc)"/>
   <xacro:property name="hardware_type"              value="$(arg hardware_type)"/>
+  <xacro:property name="sim_ignition"               value="$(arg sim_ignition)"/>
   <xacro:property name="pi_offset"                  value="0.00001"/>
   <xacro:property name="waist_limit_effort"         value="8"/>
@@ -654,8 +657,19 @@
     </xacro:if> <!-- show_gripper_bar -->
   </xacro:if> <!-- use_gripper -->
-  <xacro:include filename="$(find interbotix_xsarm_descriptions)/urdf/control.urdf.xacro"/>
+  <xacro:include filename="$(find interbotix_arm_robot_server)/urdf/control.urdf.xacro"/>
   <xacro:include filename="$(find interbotix_xsarm_descriptions)/urdf/gazebo_configs.urdf.xacro"/>
   <xacro:if value="${hardware_type == 'gz_classic'}">
     <xacro:gazebo_configs/>
+  </xacro:if>
+  <xacro:if value="$(arg sim_ignition)">
+    <!-- Gazebo plugins -->
+    <gazebo reference="world">
+    </gazebo>
+    <gazebo>
+      <plugin filename="libign_ros2_control-system.so" name="ign_ros2_control::IgnitionROS2ControlPlugin">
+        <parameters>$(arg simulation_controllers)</parameters>
+        <controller_manager_node_name>$(arg tf_prefix)controller_manager</controller_manager_node_name>
+      </plugin>
+    </gazebo>
   </xacro:if>
   <xacro:if value="${urdf_loc != ''}">

File: interbotix_arm_robot_server/urdf/mobile_wx250s.urdf.xacro (robot description, xacro)
@@ -16,7 +16,10 @@
   <xacro:arg name="external_urdf_loc"               default=""/>
   <xacro:arg name="hardware_type"                   default="actual"/>
+  <xacro:arg name="sim_ignition"                    default="true"/>
+  <xacro:arg name="simulation_controllers"          default="" />
   <xacro:property name="mesh_directory"             value="package://interbotix_xsarm_descriptions/meshes/${robot_model}_meshes"/>
   <xacro:property name="urdf_loc"                   value="$(arg external_urdf_loc)"/>
   <xacro:property name="hardware_type"              value="$(arg hardware_type)"/>
+  <xacro:property name="sim_ignition"               value="$(arg sim_ignition)"/>
   <xacro:property name="pi_offset"                  value="0.00001"/>
   <xacro:property name="waist_limit_effort"         value="10"/>
@@ -712,8 +715,19 @@
     </xacro:if> <!-- show_gripper_bar -->
   </xacro:if> <!-- use_gripper -->
-  <xacro:include filename="$(find interbotix_xsarm_descriptions)/urdf/control.urdf.xacro"/>
+  <xacro:include filename="$(find interbotix_arm_robot_server)/urdf/control.urdf.xacro"/>
   <xacro:include filename="$(find interbotix_xsarm_descriptions)/urdf/gazebo_configs.urdf.xacro"/>
   <xacro:if value="${hardware_type == 'gz_classic'}">
     <xacro:gazebo_configs/>
+  </xacro:if>
+  <xacro:if value="$(arg sim_ignition)">
+    <!-- Gazebo plugins -->
+    <gazebo reference="world">
+    </gazebo>
+    <gazebo>
+      <plugin filename="libign_ros2_control-system.so" name="ign_ros2_control::IgnitionROS2ControlPlugin">
+        <parameters>$(arg simulation_controllers)</parameters>
+        <controller_manager_node_name>$(arg tf_prefix)controller_manager</controller_manager_node_name>
+      </plugin>
+    </gazebo>
   </xacro:if>
   <xacro:if value="${urdf_loc != ''}">

File: interbotix_arm_robot_server/urdf/px100.urdf.xacro (robot description, xacro)
@@ -16,7 +16,16 @@
   <xacro:arg name="external_urdf_loc"               default=""/>
   <xacro:arg name="hardware_type"                   default="actual"/>
+  <xacro:arg name="sim_ignition"                    default="true"/>
+  <xacro:arg name="simulation_controllers"          default="" />
+  <xacro:arg name="x"                               default="0.0"/>
+  <xacro:arg name="y"                               default="0.0"/>
+  <xacro:arg name="z"                               default="0.0"/>
+  <xacro:arg name="roll"                            default="0.0"/>
+  <xacro:arg name="pitch"                           default="0.0"/>
+  <xacro:arg name="yaw"                             default="0.0"/>
   <xacro:property name="mesh_directory"             value="package://interbotix_xsarm_descriptions/meshes/${robot_model}_meshes"/>
   <xacro:property name="urdf_loc"                   value="$(arg external_urdf_loc)"/>
   <xacro:property name="hardware_type"              value="$(arg hardware_type)"/>
+  <xacro:property name="sim_ignition"               value="$(arg sim_ignition)"/>
   <xacro:property name="pi_offset"                  value="0.00001"/>
   <xacro:property name="waist_limit_effort"         value="1"/>
@@ -51,4 +60,5 @@
       <child
         link="$(arg robot_name)/$(arg base_link_frame)"/>
+      <origin xyz="$(arg x) $(arg y) $(arg z)" rpy="$(arg roll) $(arg pitch) $(arg yaw)" />
     </joint>
   </xacro:if> <!-- use_world_frame -->
@@ -596,8 +606,19 @@
     </xacro:if> <!-- show_gripper_bar -->
   </xacro:if> <!-- use_gripper -->
-  <xacro:include filename="$(find interbotix_xsarm_descriptions)/urdf/control.urdf.xacro"/>
+  <xacro:include filename="$(find interbotix_arm_robot_server)/urdf/control.urdf.xacro"/>
   <xacro:include filename="$(find interbotix_xsarm_descriptions)/urdf/gazebo_configs.urdf.xacro"/>
   <xacro:if value="${hardware_type == 'gz_classic'}">
     <xacro:gazebo_configs/>
+  </xacro:if>
+  <xacro:if value="$(arg sim_ignition)">
+    <!-- Gazebo plugins -->
+    <gazebo reference="world">
+    </gazebo>
+    <gazebo>
+      <plugin filename="libign_ros2_control-system.so" name="ign_ros2_control::IgnitionROS2ControlPlugin">
+        <parameters>$(arg simulation_controllers)</parameters>
+        <controller_manager_node_name>$(arg tf_prefix)controller_manager</controller_manager_node_name>
+      </plugin>
+    </gazebo>
   </xacro:if>
   <xacro:if value="${urdf_loc != ''}">

File: interbotix_arm_robot_server/urdf/px150.urdf.xacro (robot description, xacro)
@@ -16,7 +16,16 @@
   <xacro:arg name="external_urdf_loc"               default=""/>
   <xacro:arg name="hardware_type"                   default="actual"/>
+  <xacro:arg name="sim_ignition"                    default="true"/>
+  <xacro:arg name="simulation_controllers"          default="" />
+  <xacro:arg name="x"                               default="0.0"/>
+  <xacro:arg name="y"                               default="0.0"/>
+  <xacro:arg name="z"                               default="0.0"/>
+  <xacro:arg name="roll"                            default="0.0"/>
+  <xacro:arg name="pitch"                           default="0.0"/>
+  <xacro:arg name="yaw"                             default="0.0"/>
   <xacro:property name="mesh_directory"             value="package://interbotix_xsarm_descriptions/meshes/${robot_model}_meshes"/>
   <xacro:property name="urdf_loc"                   value="$(arg external_urdf_loc)"/>
   <xacro:property name="hardware_type"              value="$(arg hardware_type)"/>
+  <xacro:property name="sim_ignition"               value="$(arg sim_ignition)"/>
   <xacro:property name="pi_offset"                  value="0.00001"/>
   <xacro:property name="waist_limit_effort"         value="8"/>
@@ -55,4 +64,5 @@
       <child
         link="$(arg robot_name)/$(arg base_link_frame)"/>
+      <origin xyz="$(arg x) $(arg y) $(arg z)" rpy="$(arg roll) $(arg pitch) $(arg yaw)" />
     </joint>
   </xacro:if>
@@ -654,8 +664,19 @@
     </xacro:if> <!-- show_gripper_bar -->
   </xacro:if> <!-- use_gripper -->
-  <xacro:include filename="$(find interbotix_xsarm_descriptions)/urdf/control.urdf.xacro"/>
+  <xacro:include filename="$(find interbotix_arm_robot_server)/urdf/control.urdf.xacro"/>
   <xacro:include filename="$(find interbotix_xsarm_descriptions)/urdf/gazebo_configs.urdf.xacro"/>
   <xacro:if value="${hardware_type == 'gz_classic'}">
     <xacro:gazebo_configs/>
+  </xacro:if>
+  <xacro:if value="$(arg sim_ignition)">
+    <!-- Gazebo plugins -->
+    <gazebo reference="world">
+    </gazebo>
+    <gazebo>
+      <plugin filename="libign_ros2_control-system.so" name="ign_ros2_control::IgnitionROS2ControlPlugin">
+        <parameters>$(arg simulation_controllers)</parameters>
+        <controller_manager_node_name>$(arg tf_prefix)controller_manager</controller_manager_node_name>
+      </plugin>
+    </gazebo>
   </xacro:if>
   <xacro:if value="${urdf_loc != ''}">

File: interbotix_arm_robot_server/urdf/rx150.urdf.xacro (robot description, xacro)
@@ -13,10 +13,19 @@
   <xacro:arg name="show_gripper_bar"                default="true"/>
   <xacro:arg name="show_gripper_fingers"            default="true"/>
-  <xacro:arg name="use_world_frame"                 default="false"/>
+  <xacro:arg name="use_world_frame"                 default="true"/>
   <xacro:arg name="external_urdf_loc"               default=""/>
   <xacro:arg name="hardware_type"                   default="actual"/>
+  <xacro:arg name="sim_ignition"                    default="true"/>
+  <xacro:arg name="simulation_controllers"          default="" />
+  <xacro:arg name="x"                               default="0.0"/>
+  <xacro:arg name="y"                               default="0.0"/>
+  <xacro:arg name="z"                               default="0.0"/>
+  <xacro:arg name="roll"                            default="0.0"/>
+  <xacro:arg name="pitch"                           default="0.0"/>
+  <xacro:arg name="yaw"                             default="0.0"/>
   <xacro:property name="mesh_directory"             value="package://interbotix_xsarm_descriptions/meshes/${robot_model}_meshes"/>
   <xacro:property name="urdf_loc"                   value="$(arg external_urdf_loc)"/>
   <xacro:property name="hardware_type"              value="$(arg hardware_type)"/>
+  <xacro:property name="sim_ignition"               value="$(arg sim_ignition)"/>
   <xacro:property name="pi_offset"                  value="0.00001"/>
   <xacro:property name="waist_limit_effort"         value="8"/>
@@ -55,4 +64,5 @@
       <child
         link="$(arg robot_name)/$(arg base_link_frame)"/>
+      <origin xyz="$(arg x) $(arg y) $(arg z)" rpy="$(arg roll) $(arg pitch) $(arg yaw)" />
     </joint>
   </xacro:if> <!-- use_world_frame -->
@@ -654,8 +664,19 @@
     </xacro:if> <!-- show_gripper_bar -->
   </xacro:if> <!-- use_gripper -->
-  <xacro:include filename="$(find interbotix_xsarm_descriptions)/urdf/control.urdf.xacro"/>
+  <xacro:include filename="$(find interbotix_arm_robot_server)/urdf/control.urdf.xacro"/>
   <xacro:include filename="$(find interbotix_xsarm_descriptions)/urdf/gazebo_configs.urdf.xacro"/>
   <xacro:if value="${hardware_type == 'gz_classic'}">
     <xacro:gazebo_configs/>
+  </xacro:if>
+  <xacro:if value="$(arg sim_ignition)">
+    <!-- Gazebo plugins -->
+    <gazebo reference="world">
+    </gazebo>
+    <gazebo>
+      <plugin filename="libign_ros2_control-system.so" name="ign_ros2_control::IgnitionROS2ControlPlugin">
+        <parameters>$(arg simulation_controllers)</parameters>
+        <controller_manager_name>controller_manager</controller_manager_name>
+      </plugin>
+    </gazebo>
   </xacro:if>
   <xacro:if value="${urdf_loc != ''}">

File: interbotix_arm_robot_server/urdf/rx200.urdf.xacro (robot description, xacro)
@@ -16,7 +16,16 @@
   <xacro:arg name="external_urdf_loc"               default=""/>
   <xacro:arg name="hardware_type"                   default="actual"/>
+  <xacro:arg name="sim_ignition"                    default="true"/>
+  <xacro:arg name="simulation_controllers"          default="" />
+  <xacro:arg name="x"                               default="0.0"/>
+  <xacro:arg name="y"                               default="0.0"/>
+  <xacro:arg name="z"                               default="0.0"/>
+  <xacro:arg name="roll"                            default="0.0"/>
+  <xacro:arg name="pitch"                           default="0.0"/>
+  <xacro:arg name="yaw"                             default="0.0"/>
   <xacro:property name="mesh_directory"             value="package://interbotix_xsarm_descriptions/meshes/${robot_model}_meshes"/>
   <xacro:property name="urdf_loc"                   value="$(arg external_urdf_loc)"/>
   <xacro:property name="hardware_type"              value="$(arg hardware_type)"/>
+  <xacro:property name="sim_ignition"               value="$(arg sim_ignition)"/>
   <xacro:property name="pi_offset"                  value="0.00001"/>
   <xacro:property name="waist_limit_effort"         value="8"/>
@@ -55,4 +64,5 @@
       <child
         link="$(arg robot_name)/$(arg base_link_frame)"/>
+      <origin xyz="$(arg x) $(arg y) $(arg z)" rpy="$(arg roll) $(arg pitch) $(arg yaw)" />
     </joint>
   </xacro:if> <!-- use_world_frame -->
@@ -654,8 +664,19 @@
     </xacro:if> <!-- show_gripper_bar -->
   </xacro:if> <!-- use_gripper -->
-  <xacro:include filename="$(find interbotix_xsarm_descriptions)/urdf/control.urdf.xacro"/>
+  <xacro:include filename="$(find interbotix_arm_robot_server)/urdf/control.urdf.xacro"/>
   <xacro:include filename="$(find interbotix_xsarm_descriptions)/urdf/gazebo_configs.urdf.xacro"/>
   <xacro:if value="${hardware_type == 'gz_classic'}">
     <xacro:gazebo_configs/>
+  </xacro:if>
+  <xacro:if value="$(arg sim_ignition)">
+    <!-- Gazebo plugins -->
+    <gazebo reference="world">
+    </gazebo>
+    <gazebo>
+      <plugin filename="libign_ros2_control-system.so" name="ign_ros2_control::IgnitionROS2ControlPlugin">
+        <parameters>$(arg simulation_controllers)</parameters>
+        <controller_manager_node_name>$(arg tf_prefix)controller_manager</controller_manager_node_name>
+      </plugin>
+    </gazebo>
   </xacro:if>
   <xacro:if value="${urdf_loc != ''}">

File: interbotix_arm_robot_server/urdf/vx250.urdf.xacro (robot description, xacro)
@@ -16,7 +16,16 @@
   <xacro:arg name="external_urdf_loc"               default=""/>
   <xacro:arg name="hardware_type"                   default="actual"/>
+  <xacro:arg name="sim_ignition"                    default="true"/>
+  <xacro:arg name="simulation_controllers"          default="" />
+  <xacro:arg name="x"                               default="0.0"/>
+  <xacro:arg name="y"                               default="0.0"/>
+  <xacro:arg name="z"                               default="0.0"/>
+  <xacro:arg name="roll"                            default="0.0"/>
+  <xacro:arg name="pitch"                           default="0.0"/>
+  <xacro:arg name="yaw"                             default="0.0"/>
   <xacro:property name="mesh_directory"             value="package://interbotix_xsarm_descriptions/meshes/${robot_model}_meshes"/>
   <xacro:property name="urdf_loc"                   value="$(arg external_urdf_loc)"/>
   <xacro:property name="hardware_type"              value="$(arg hardware_type)"/>
+  <xacro:property name="sim_ignition"               value="$(arg sim_ignition)"/>
   <xacro:property name="pi_offset"                  value="0.00001"/>
   <xacro:property name="waist_limit_effort"         value="10"/>
@@ -55,4 +64,5 @@
       <child
         link="$(arg robot_name)/$(arg base_link_frame)"/>
+      <origin xyz="$(arg x) $(arg y) $(arg z)" rpy="$(arg roll) $(arg pitch) $(arg yaw)" />
     </joint>
   </xacro:if> <!-- use_world_frame -->
@@ -654,8 +664,19 @@
     </xacro:if> <!-- show_gripper_bar -->
   </xacro:if> <!-- use_gripper -->
-  <xacro:include filename="$(find interbotix_xsarm_descriptions)/urdf/control.urdf.xacro"/>
+  <xacro:include filename="$(find interbotix_arm_robot_server)/urdf/control.urdf.xacro"/>
   <xacro:include filename="$(find interbotix_xsarm_descriptions)/urdf/gazebo_configs.urdf.xacro"/>
   <xacro:if value="${hardware_type == 'gz_classic'}">
     <xacro:gazebo_configs/>
+  </xacro:if>
+  <xacro:if value="$(arg sim_ignition)">
+    <!-- Gazebo plugins -->
+    <gazebo reference="world">
+    </gazebo>
+    <gazebo>
+      <plugin filename="libign_ros2_control-system.so" name="ign_ros2_control::IgnitionROS2ControlPlugin">
+        <parameters>$(arg simulation_controllers)</parameters>
+        <controller_manager_node_name>$(arg tf_prefix)controller_manager</controller_manager_node_name>
+      </plugin>
+    </gazebo>
   </xacro:if>
   <xacro:if value="${urdf_loc != ''}">
