Commit message: locobot working

File: interbotix_rover_robot_server/urdf/locobot.urdf.xacro (robot description, xacro)
@@ -3,19 +3,16 @@
   <xacro:arg name="arm_model"             default=""/>
   <xacro:arg name="robot_model"           default=""/>
-  <xacro:arg name="base_model"            default=""/>
   <xacro:arg name="robot_name"            default=""/>
-  <xacro:arg name="show_lidar"            default="true"/>
+  <xacro:arg name="base_model"            default="create3"/>
+  <xacro:arg name="use_lidar"             default="true"/>
+  <xacro:arg name="show_ar_tag"           default="true"/>
   <xacro:arg name="show_gripper_bar"      default="true"/>
   <xacro:arg name="show_gripper_fingers"  default="true"/>
   <xacro:arg name="external_urdf_loc"     default=""/>
-  <!-- rgbd camera arguments -->
-  <xacro:arg name="camera1_gazebo" default="False"/>
-  <xacro:arg name="camera1_link_x" default="0.0"/>
-  <xacro:arg name="camera1_link_y" default="0.0"/>
-  <xacro:arg name="camera1_link_z" default="0.0"/>
-  <xacro:arg name="camera1_link_roll" default="0.0"/>
-  <xacro:arg name="camera1_link_pitch" default="0.0"/>
-  <xacro:arg name="camera1_link_yaw" default="0.0"/>
+  <xacro:arg name="use_gripper"           default="true"/>
+  <xacro:arg name="hardware_type"         default="actual"/>
+  <xacro:property name="hardware_type"    value="$(arg hardware_type)"/>
   <xacro:property name="arm_type"         value="$(arg arm_model)"/>
+  <xacro:property name="robot_name"       value="$(arg robot_name)"/>
   <xacro:property name="base_type"        value="$(arg base_model)"/>
   <xacro:property name="urdf_loc"         value="$(arg external_urdf_loc)"/>
@@ -25,5 +22,5 @@
   </xacro:if>
   <material name="interbotix_black">
-    <texture filename="package://interbotix_xslocobot_descriptions/meshes/interbotix_black.png"/>
+    <texture filename="package://interbotix_common_sim/media/materials/textures/interbotix_black.png"/>
   </material>
   <xacro:include filename="$(find interbotix_xslocobot_descriptions)/urdf/plate.urdf.xacro" />
@@ -33,5 +30,4 @@
   <xacro:include filename="$(find interbotix_xslocobot_descriptions)/urdf/camera_tower.urdf.xacro" />
   <xacro:include filename="$(find interbotix_xslocobot_descriptions)/urdf/pan_and_tilt.urdf.xacro" />
-  <link name="$(arg robot_name)/base_footprint"/>
   <xacro:if value="${arm_type == 'mobile_wx250s'}">
     <xacro:property name="camera_tower_size" value="large"/>
@@ -51,9 +47,19 @@
   <xacro:if value="${base_type == 'kobuki'}">
     <xacro:plate>
-      <origin rpy="0 0 0" xyz="0.0 0 0.08825"/>
+      <origin
+        rpy="0 0 0"
+        xyz="0.0 0 0.08825"/>
       <inertial>
-        <origin rpy="0 0 0" xyz="0.050816 0 0.00475"/>
+        <origin
+          rpy="0 0 0"
+          xyz="0.050816 0 0.00475"/>
         <mass value="0.571995"/>
-        <inertia ixx="0.003115" ixy="0" ixz="0" iyy="0.001813" iyz="0" izz="0.004919"/>
+        <inertia
+          ixx="0.003115"
+          ixy="0"
+          ixz="0"
+          iyy="0.001813"
+          iyz="0"
+          izz="0.004919"/>
       </inertial>
     </xacro:plate>
@@ -61,9 +67,19 @@
   <xacro:if value="${base_type == 'create3'}">
     <xacro:plate>
-      <origin rpy="0 0 0" xyz="0 0 0.0934"/>
+      <origin
+        rpy="0 0 0"
+        xyz="0 0 0.0934"/>
       <inertial>
-        <origin rpy="0 0 0" xyz="-0.005869 0 4.67E-03"/>
+        <origin
+          rpy="0 0 0"
+          xyz="-0.005869 0 4.67E-03"/>
         <mass value="0.807674"/>
-        <inertia ixx="5.27E-03" ixy="0" ixz="0" iyy="3.27E-03" iyz="0" izz="8.54E-03"/>
+        <inertia
+          ixx="5.27E-03"
+          ixy="0"
+          ixz="0"
+          iyy="3.27E-03"
+          iyz="0"
+          izz="8.54E-03"/>
       </inertial>
     </xacro:plate>
@@ -76,10 +92,14 @@
       <xacro:if value="${base_type == 'kobuki'}">
         <xacro:arm_cradle>
-          <origin rpy="0 0 0" xyz="0.0215 0 0.1195"/>
+          <origin
+            rpy="0 0 0"
+            xyz="0.0215 0 0.1195"/>
         </xacro:arm_cradle>
       </xacro:if> <!-- base_type == 'kobuki' -->
       <xacro:if value="${base_type == 'create3'}">
         <xacro:arm_cradle>
-          <origin rpy="0 0 0" xyz="0.037943 0 0.139"/>
+          <origin
+            rpy="0 0 0"
+            xyz="0.037943 0 0.139"/>
         </xacro:arm_cradle>
       </xacro:if> <!-- base_type == 'create3' -->
@@ -89,10 +109,14 @@
   <xacro:if value="${base_type == 'kobuki'}">
     <xacro:battery>
-      <origin rpy="0 0 0" xyz="-0.007 0 0.0125"/>
+      <origin
+        rpy="0 0 0"
+        xyz="-0.007 0 0.0125"/>
     </xacro:battery>
   </xacro:if> <!-- base_type == 'kobuki' -->
   <xacro:if value="${base_type == 'create3'}">
     <xacro:battery>
-      <origin rpy="0 0 0" xyz="-0.0345 0 0.010763"/>
+      <origin
+        rpy="0 0 0"
+        xyz="-0.0345 0 0.010763"/>
     </xacro:battery>
   </xacro:if> <!-- base_type == 'create3' -->
@@ -101,9 +125,19 @@
     <xacro:if value="${camera_tower_size == 'large'}">
       <xacro:camera_tower>
-        <origin rpy="0 0 0" xyz="-0.023997 -0.000044 0.08823"/>
-        <inertial>
-          <origin rpy="0 0 0" xyz="-0.0372211000 -0.0026114300 0.1744600000"/>
+        <origin
+          rpy="0 0 0"
+          xyz="-0.023997 -0.000044 0.08823"/>
+        <inertial>
+          <origin
+            rpy="0 0 0"
+            xyz="-0.0372211000 -0.0026114300 0.1744600000"/>
           <mass value="2.366224"/>
-          <inertia ixx="0.0628500000" ixy="0.0002152000" ixz="0.0065630000" iyy="0.0546000000" iyz="-0.0004738000" izz="0.0179300000"/>
+          <inertia
+            ixx="0.0628500000"
+            ixy="0.0002152000"
+            ixz="0.0065630000"
+            iyy="0.0546000000"
+            iyz="-0.0004738000"
+            izz="0.0179300000"/>
         </inertial>
       </xacro:camera_tower>
@@ -111,9 +145,19 @@
     <xacro:if value="${camera_tower_size == 'small'}">
       <xacro:camera_tower>
-        <origin rpy="0 0 0" xyz="-0.023997 -0.000044 0.08823"/>
-        <inertial>
-          <origin rpy="0 0 0" xyz="-0.0357703000 -0.0027068600 0.1560470000"/>
+        <origin
+          rpy="0 0 0"
+          xyz="-0.023997 -0.000044 0.08823"/>
+        <inertial>
+          <origin
+            rpy="0 0 0"
+            xyz="-0.0357703000 -0.0027068600 0.1560470000"/>
           <mass value="2.282808"/>
-          <inertia ixx="0.0461600000" ixy="0.0002062000" ixz="0.0052560000" iyy="0.0384200000" iyz="-0.0003600000" izz="0.0169600000"/>
+          <inertia
+            ixx="0.0461600000"
+            ixy="0.0002062000"
+            ixz="0.0052560000"
+            iyy="0.0384200000"
+            iyz="-0.0003600000"
+            izz="0.0169600000"/>
         </inertial>
       </xacro:camera_tower>
@@ -123,9 +167,19 @@
     <xacro:if value="${camera_tower_size == 'large'}">
       <xacro:camera_tower>
-        <origin rpy="0 0 0" xyz="-0.048271 0 0.10087"/>
-        <inertial>
-          <origin rpy="0 0 0" xyz="-0.025958 -0.003319 0.205872"/>
+        <origin
+          rpy="0 0 0"
+          xyz="-0.048271 0 0.10087"/>
+        <inertial>
+          <origin
+            rpy="0 0 0"
+            xyz="-0.025958 -0.003319 0.205872"/>
           <mass value="2.514064"/>
-          <inertia ixx="7.61E-02" ixy="1.47E-04" ixz="7.04E-03" iyy="6.71E-02" iyz="-9.41E-04" izz="1.95E-02"/>
+          <inertia
+            ixx="7.61E-02"
+            ixy="1.47E-04"
+            ixz="7.04E-03"
+            iyy="6.71E-02"
+            iyz="-9.41E-04"
+            izz="1.95E-02"/>
         </inertial>
       </xacro:camera_tower>
@@ -133,9 +187,19 @@
     <xacro:if value="${camera_tower_size == 'small'}">
       <xacro:camera_tower>
-        <origin rpy="0 0 0" xyz="-0.048271 0 0.10087"/>
-        <inertial>
-          <origin rpy="0 0 0" xyz="-0.024689 -0.003432 0.185408"/>
+        <origin
+          rpy="0 0 0"
+          xyz="-0.048271 0 0.10087"/>
+        <inertial>
+          <origin
+            rpy="0 0 0"
+            xyz="-0.024689 -0.003432 0.185408"/>
           <mass value="2.430647"/>
-          <inertia ixx="5.63E-02" ixy="1.37E-04" ixz="5.75E-03" iyy="4.78E-02" iyz="-7.70E-04" izz="1.86E-02"/>
+          <inertia
+            ixx="5.63E-02"
+            ixy="1.37E-04"
+            ixz="5.75E-03"
+            iyy="4.78E-02"
+            iyz="-7.70E-04"
+            izz="1.86E-02"/>
         </inertial>
       </xacro:camera_tower>
@@ -146,10 +210,14 @@
     <xacro:if value="${camera_tower_size == 'large'}">
       <xacro:pan_and_tilt>
-        <origin rpy="0 0 0" xyz="0.047228 0 0.44425"/>
+        <origin
+          rpy="0 0 0"
+          xyz="0.047228 0 0.44425"/>
       </xacro:pan_and_tilt>
     </xacro:if> <!-- base_type == 'kobuki' && camera_tower_size == 'large' -->
     <xacro:if value="${camera_tower_size == 'small'}">
       <xacro:pan_and_tilt>
-        <origin rpy="0 0 0" xyz="0.047228 0 0.38425"/>
+        <origin
+          rpy="0 0 0"
+          xyz="0.047228 0 0.38425"/>
       </xacro:pan_and_tilt>
     </xacro:if> <!-- base_type == 'kobuki' && camera_tower_size == 'small' -->
@@ -158,24 +226,32 @@
     <xacro:if value="${camera_tower_size == 'large'}">
       <xacro:pan_and_tilt>
-        <origin rpy="0 0 0" xyz="0.061228 0 0.462"/>
+        <origin
+          rpy="0 0 0"
+          xyz="0.061228 0 0.462"/>
       </xacro:pan_and_tilt>
     </xacro:if> <!-- base_type == 'create3' && camera_tower_size == 'large' -->
     <xacro:if value="${camera_tower_size == 'small'}">
       <xacro:pan_and_tilt>
-        <origin rpy="0 0 0" xyz="0.061228 0 0.402"/>
+        <origin
+          rpy="0 0 0"
+          xyz="0.061228 0 0.402"/>
       </xacro:pan_and_tilt>
     </xacro:if> <!-- base_type == 'create3' && camera_tower_size == 'small' -->
   </xacro:if> <!-- base_type == 'create3' -->
   <!-- ********************************** Lidar **********************************  -->
-  <xacro:if value="$(arg show_lidar)">
+  <xacro:if value="$(arg use_lidar)">
     <xacro:if value="${base_type == 'kobuki'}">
       <xacro:if value="${camera_tower_size == 'large'}">
         <xacro:lidar>
-          <origin rpy="0 0 0" xyz="-0.074 0 0.44425"/>
+          <origin
+            rpy="0 0 0"
+            xyz="-0.074 0 0.44425"/>
         </xacro:lidar>
       </xacro:if> <!-- base_type == 'kobuki' && camera_tower_size == 'large' -->
       <xacro:if value="${camera_tower_size == 'small'}">
         <xacro:lidar>
-          <origin rpy="0 0 0" xyz="-0.074 0 0.38425"/>
+          <origin
+            rpy="0 0 0"
+            xyz="-0.074 0 0.38425"/>
         </xacro:lidar>
       </xacro:if> <!-- base_type == 'kobuki' && camera_tower_size == 'small' -->
@@ -184,24 +260,17 @@
       <xacro:if value="${camera_tower_size == 'large'}">
         <xacro:lidar>
-          <origin rpy="0 0 0" xyz="-0.066095 0 0.462"/>
-        </xacro:lidar>
-      </xacro:if> <!-- base_type == 'create3' && camera_tower_size == 'large' -->
+          <origin
+            rpy="0 0 0"
+            xyz="-0.066095 0 0.462"/>
+        </xacro:lidar>
+      </xacro:if> <!-- base_type == 'create3' && camera_tower_size == 'large'libgazebo_ros_ray_sensor -->
       <xacro:if value="${camera_tower_size == 'small'}">
         <xacro:lidar>
-          <origin rpy="0 0 0" xyz="-0.066095 0 0.402"/>
+          <origin
+            rpy="0 0 0"
+            xyz="-0.066095 0 0.402"/>
         </xacro:lidar>
       </xacro:if> <!-- base_type == 'create3' && camera_tower_size == 'small' -->
     </xacro:if> <!-- base_type == 'create3' -->
-  </xacro:if> <!-- show_lidar -->
-  <!-- simulated rgbd camera include -->
-  <xacro:if value="$(arg camera1_gazebo)">
-    <xacro:include filename="$(find scene_perception)/urdf/rgbd_camera_macro.xacro"/>
-    <xacro:rgbd_camera_gazebo camera_name="camera1"/>
-    <joint name="camera1_joint" type="fixed">
-      <parent link="world"/>
-      <child link="camera1_link"/>
-      <origin xyz="$(arg camera1_link_x) $(arg camera1_link_y) $(arg camera1_link_z)"
-        rpy="$(arg camera1_link_roll) $(arg camera1_link_pitch) $(arg camera1_link_yaw)" />
-    </joint>
-  </xacro:if>
+  </xacro:if> <!-- use_lidar -->
 </robot>
